File: HARDWARE/Serial_NID/_saved_Serial_NID.sch (KiCad schematic (older format))
At the start: 22 parts, among them J1 CONN_01X04, J2 CONN_01X07, J3 USB_OTG, SW1 SW_PUSH, U1 TPS2550, U2 STM32L011Gx, U3 FT230XQ

Commit message: updated pcb
Parts:
- added R6: R, ZF_footprints:ZF_SMD_NonPol_0402, symbol R
- D1: renamed from D?; footprint (none) -> ZF_footprints:ZF_SMD_NonPol_0402
- J3: footprint ZF:JW_USBMICROB_SMT -> ZF_footprints:JW_USBMICROB_SMT
- R7: renamed from R?; footprint (none) -> ZF_footprints:ZF_SMD_NonPol_0402
- SW1: footprint ZF:ZF_SW_Momentary_SideMtg -> ZF_footprints:ZF_SW_Momentary_SideMtg
- U2: footprint ZF:ZF_IC_UFQFPN28-050 -> ZF_footprints:ZF_IC_UFQFPN28-050
Connections:
- net +5V: now also R6.1; no longer U1.3 (EN)
- net FAULT: now also U2.13 (PA7_5V/MOSI)
- net EN: now reaches U2.14 (PB0_5V/TIM2_CH2/3)
- net EN: now also U1.3 (EN), R6.2
Other:
- moved on the sheet: C1
Changed lines of the file:
@@
 F 0 "U2" H 5400 1875 60  0000 C CNN
 F 1 "STM32L011Gx" H 5400 2750 60  0000 C CNN
-F 2 "ZF:ZF_IC_UFQFPN28-050" H 5400 2300 60  0001 C CNN
+F 2 "ZF_footprints:ZF_IC_UFQFPN28-050" H 5400 2300 60  0001 C CNN
 F 3 "" H 5400 2300 60  0001 C CNN
 	1    5400 2300
@@
 F 0 "SW1" H 1100 1010 50  0000 C CNN
 F 1 "SW_PUSH" H 950 820 50  0000 C CNN
-F 2 "ZF:ZF_SW_Momentary_SideMtg" H 950 900 50  0001 C CNN
+F 2 "ZF_footprints:ZF_SW_Momentary_SideMtg" H 950 900 50  0001 C CNN
 F 3 "" H 950 900 50  0000 C CNN
 	1    950  900
@@
 F 0 "J3" H 6700 5500 50  0000 L CNN
 F 1 "USB_OTG" H 6700 5400 50  0000 L CNN
-F 2 "ZF:JW_USBMICROB_SMT" H 7050 5000 50  0001 C CNN
+F 2 "ZF_footprints:JW_USBMICROB_SMT" H 7050 5000 50  0001 C CNN
 F 3 "" H 7050 5000 50  0001 C CNN
 	1    6900 5050
@@
 L +5V #PWR016
 U 1 1 594446BF
-P 2250 5000
-F 0 "#PWR016" H 2250 4850 50  0001 C CNN
-F 1 "+5V" H 2250 5140 50  0000 C CNN
-F 2 "" H 2250 5000 50  0001 C CNN
-F 3 "" H 2250 5000 50  0001 C CNN
-	1    2250 5000
+P 1900 5000
+F 0 "#PWR016" H 1900 4850 50  0001 C CNN
+F 1 "+5V" H 1900 5140 50  0000 C CNN
+F 2 "" H 1900 5000 50  0001 C CNN
+F 3 "" H 1900 5000 50  0001 C CNN
+	1    1900 5000
 	1    0    0    -1
 $EndComp
@@
 $EndComp
 Wire Wire Line
-	2250 5000 2250 5250
-Wire Wire Line
-	2250 5250 2600 5250
+	1900 5000 1900 5250
 Wire Wire Line
 	4000 5000 4000 5250
@@
 L C C1
 U 1 1 594449B9
-P 2250 5400
-F 0 "C1" H 2275 5500 50  0000 L CNN
-F 1 "C" H 2275 5300 50  0000 L CNN
-F 2 "ZF_footprints:ZF_SMD_NonPol_0402_cap" H 2288 5250 50  0001 C CNN
-F 3 "" H 2250 5400 50  0001 C CNN
-	1    2250 5400
+P 1900 5400
+F 0 "C1" H 1925 5500 50  0000 L CNN
+F 1 "C" H 1925 5300 50  0000 L CNN
+F 2 "ZF_footprints:ZF_SMD_NonPol_0402_cap" H 1938 5250 50  0001 C CNN
+F 3 "" H 1900 5400 50  0001 C CNN
+	1    1900 5400
 	-1   0    0    1
 $EndComp
@@
 L GND #PWR018
 U 1 1 59444A62
-P 2350 5800
-F 0 "#PWR018" H 2350 5550 50  0001 C CNN
-F 1 "GND" H 2350 5650 50  0000 C CNN
-F 2 "" H 2350 5800 50  0001 C CNN
-F 3 "" H 2350 5800 50  0001 C CNN
-	1    2350 5800
-	1    0    0    -1
-$EndComp
-Wire Wire Line
-	2600 5400 2450 5400
-Wire Wire Line
-	2450 5400 2450 5700
-Wire Wire Line
-	2450 5700 2250 5700
-Wire Wire Line
-	2350 5700 2350 5800
-Wire Wire Line
-	2250 5700 2250 5550
-Connection ~ 2350 5700
-Wire Wire Line
-	2600 5550 2550 5550
-Wire Wire Line
-	2550 5550 2550 5250
-Connection ~ 2550 5250
+P 2000 5800
+F 0 "#PWR018" H 2000 5550 50  0001 C CNN
+F 1 "GND" H 2000 5650 50  0000 C CNN
+F 2 "" H 2000 5800 50  0001 C CNN
+F 3 "" H 2000 5800 50  0001 C CNN
+	1    2000 5800
+	1    0    0    -1
+$EndComp
+Wire Wire Line
+	1900 5700 2450 5700
+Wire Wire Line
+	2000 5700 2000 5800
+Wire Wire Line
+	1900 5700 1900 5550
+Connection ~ 2000 5700
+Wire Wire Line
+	2200 5550 2600 5550
 $Comp
 L R R3
@@
 Wire Wire Line
 	4950 5700 4950 5900
-Text GLabel 4350 5550 2    60   Input ~ 0
+Text GLabel 4350 5550 2    60   Output ~ 0
 FAULT
 Wire Wire Line
@@
 	4200 2450 4050 2450
 $Comp
-L LED D?
+L LED D1
 U 1 1 59472070
 P 2000 1250
-F 0 "D?" H 2000 1350 50  0000 C CNN
+F 0 "D1" H 2000 1350 50  0000 C CNN
 F 1 "LED" H 2000 1150 50  0000 C CNN
-F 2 "" H 2000 1250 50  0001 C CNN
+F 2 "ZF_footprints:ZF_SMD_NonPol_0402" H 2000 1250 50  0001 C CNN
 F 3 "" H 2000 1250 50  0001 C CNN
 	1    2000 1250
@@
 $EndComp
 $Comp
-L R R?
+L R R7
 U 1 1 594721A1
 P 2550 1250
-F 0 "R?" V 2630 1250 50  0000 C CNN
+F 0 "R7" V 2630 1250 50  0000 C CNN
 F 1 "R" V 2550 1250 50  0000 C CNN
-F 2 "" V 2480 1250 50  0001 C CNN
+F 2 "ZF_footprints:ZF_SMD_NonPol_0402" V 2480 1250 50  0001 C CNN
 F 3 "" H 2550 1250 50  0001 C CNN
 	1    2550 1250
@@
 $EndComp
 $Comp
-L GND #PWR?
+L GND #PWR026
 U 1 1 59472434
 P 1700 1500
-F 0 "#PWR?" H 1700 1250 50  0001 C CNN
+F 0 "#PWR026" H 1700 1250 50  0001 C CNN
 F 1 "GND" H 1700 1350 50  0000 C CNN
 F 2 "" H 1700 1500 50  0001 C CNN
@@
 Wire Wire Line
 	4000 2150 4200 2150
+Text GLabel 4000 3200 0    60   Input ~ 0
+FAULT
+Wire Wire Line
+	4000 3200 4200 3200
+Wire Wire Line
+	2600 5400 2450 5400
+Wire Wire Line
+	2450 5400 2450 5700
+$Comp
+L R R6
+U 1 1 59472E4E
+P 2200 5400
+F 0 "R6" V 2280 5400 50  0000 C CNN
+F 1 "R" V 2200 5400 50  0000 C CNN
+F 2 "ZF_footprints:ZF_SMD_NonPol_0402" V 2130 5400 50  0001 C CNN
+F 3 "" H 2200 5400 50  0001 C CNN
+	1    2200 5400
+	1    0    0    -1
+$EndComp
+Connection ~ 2200 5250
+Wire Wire Line
+	1900 5250 2600 5250
+Text GLabel 2200 5900 3    60   Input ~ 0
+EN
+Wire Wire Line
+	2200 5550 2200 5900
+Text GLabel 4000 3350 0    60   Output ~ 0
+EN
+Wire Wire Line
+	4200 3350 4000 3350
 $EndSCHEMATC
