File: HARDWARE/Serial_NID/Serial_NID.sch (KiCad schematic (older format))
At the start: 15 parts, among them J1 CONN_01X04, J2 CONN_01X07, J3 USB_OTG, SW1 SW_PUSH, U1 TPS2550, U2 STM32L011Gx, U3 FT230XQ

Commit message: updated pcb
Parts:
- added C6, C7, C8: C, ZF_footprints:ZF_SMD_NonPol_0402_cap, symbol C
- added D1: LED, ZF_footprints:ZF_SMD_NonPol_0402, symbol LED
- added R4, R5, R6, R7: R, ZF_footprints:ZF_SMD_NonPol_0402, symbol R
- C1, C2, C3, C4, C5: footprint Capacitors_SMD:C_0603_HandSoldering -> ZF_footprints:ZF_SMD_NonPol_0402_cap
- J3: footprint Connectors:USB_Micro-B -> ZF:JW_USBMICROB_SMT
- R1, R2, R3: footprint Resistors_SMD:R_0603 -> ZF_footprints:ZF_SMD_NonPol_0402
- SW1: footprint (none) -> ZF:ZF_SW_Momentary_SideMtg
- U2: footprint Housings_DFN_QFN:UQFN-28-1EP_4x4mm_Pitch0.4mm -> ZF:ZF_IC_UFQFPN28-050
Connections:
- net +3V3: now also U3.1 (VCCIO), U3.9 (~RESET)
- net +5V: now also C8.1, R6.1; no longer U1.3 (EN)
- net FAULT: now also U2.13 (PA7_5V/MOSI)
- net GND: now also C6.1, C7.2, C8.2, D1.1 (K)
- net CBUS2: now reaches U2.10 (PA4_3V3/NSS)
- net CBUS2: now also U3.5 (CBUS2)
- net CBUS3: now reaches U2.11 (PA5_3V3/TIM2_CH1)
- net CBUS3: now also U3.14 (CBUS3)
- net EN: now reaches U2.14 (PB0_5V/TIM2_CH2/3)
- net EN: now also U1.3 (EN), R6.2
- net LED1: now reaches U2.6 (PA0_3V3/TIM2_CH1)
- net LED1: now also R7.2
- net CBUS0: now reaches U2.8 (PA2_3V3/TIM2_CH3/TIM21_CH1)
- net CBUS0: now also U3.12 (CBUS0)
- net CBUS1: now reaches U2.9 (PA3_5V/TIM2_CH4/TIM21_CH2)
- net CBUS1: now also U3.11 (CBUS1)
- net at J3.2 (D-): now also C7.1, R5.2; no longer U3.7 (USBDM)
- net at J3.3 (D+): now also C6.2, R4.2; no longer U3.6 (USBDP)
- new net: R5.1, U3.6 (USBDP)
- new net: R4.1, U3.7 (USBDM)
- new net: D1.2 (A), R7.1
Other:
- moved on the sheet: C1, C3, J1, J2, J3

Commit message: fixed pcb
Parts:
- added C10, C9: C, ZF_footprints:ZF_SMD_NonPol_0402_cap, symbol C
- J1: footprint Connectors_JST:JST_GH_SM04B-GHS-TB_04x1.25mm_Angled -> ZF_footprints:ZF_CONN_JST_GH
- J2: footprint Connectors_JST:JST_GH_SM07B-GHS-TB_07x1.25mm_Angled -> ZF_footprints:ZF_CONN_JST_GH_7POS
- J3: footprint ZF:JW_USBMICROB_SMT -> ZF_footprints:ZF_CONN_USB-MICRO-B-SMD-holes
- SW1: footprint ZF:ZF_SW_Momentary_SideMtg -> ZF_footprints:ZF_SW_Momentary_SideMtg
- U2: footprint ZF:ZF_IC_UFQFPN28-050 -> ZF_footprints:ZF_IC_UFQFPN28-050
- U3: footprint Housings_DFN_QFN:QFN-16-1EP_3x3mm_Pitch0.5mm -> Housings_DFN_QFN:QFN-16-1EP_4x4mm_Pitch0.65mm
Connections:
- net +5V: now also C10.1, C9.1
- net GND: now also C10.2, C9.2
- net USART2_RX: now also U2.28 (PB7_5V/TIM2_CH4); no longer U2.27 (PB6_5V/TIM2_CH3)
- net USART2_TX: now also U2.27 (PB6_5V/TIM2_CH3); no longer U2.28 (PB7_5V/TIM2_CH4)
Changed lines of the file:
@@
 F 0 "U2" H 5400 1875 60  0000 C CNN
 F 1 "STM32L011Gx" H 5400 2750 60  0000 C CNN
-F 2 "ZF:ZF_IC_UFQFPN28-050" H 5400 2300 60  0001 C CNN
+F 2 "ZF_footprints:ZF_IC_UFQFPN28-050" H 5400 2300 60  0001 C CNN
 F 3 "" H 5400 2300 60  0001 C CNN
 	1    5400 2300
@@
 F 0 "SW1" H 1100 1010 50  0000 C CNN
 F 1 "SW_PUSH" H 950 820 50  0000 C CNN
-F 2 "ZF:ZF_SW_Momentary_SideMtg" H 950 900 50  0001 C CNN
+F 2 "ZF_footprints:ZF_SW_Momentary_SideMtg" H 950 900 50  0001 C CNN
 F 3 "" H 950 900 50  0000 C CNN
 	1    950  900
@@
 F 0 "J1" H 1400 2650 50  0000 C CNN
 F 1 "CONN_01X04" V 1500 2400 50  0000 C CNN
-F 2 "Connectors_JST:JST_GH_SM04B-GHS-TB_04x1.25mm_Angled" H 1400 2400 50  0001 C CNN
+F 2 "ZF_footprints:ZF_CONN_JST_GH" H 1400 2400 50  0001 C CNN
 F 3 "" H 1400 2400 50  0001 C CNN
 	1    1400 2400
@@
 F 0 "J2" H 1400 3750 50  0000 C CNN
 F 1 "CONN_01X07" V 1500 3350 50  0000 C CNN
-F 2 "Connectors_JST:JST_GH_SM07B-GHS-TB_07x1.25mm_Angled" H 1400 3350 50  0001 C CNN
+F 2 "ZF_footprints:ZF_CONN_JST_GH_7POS" H 1400 3350 50  0001 C CNN
 F 3 "" H 1400 3350 50  0001 C CNN
 	1    1400 3350
@@
 F 0 "J3" H 6700 5500 50  0000 L CNN
 F 1 "USB_OTG" H 6700 5400 50  0000 L CNN
-F 2 "ZF:JW_USBMICROB_SMT" H 7050 5000 50  0001 C CNN
+F 2 "ZF_footprints:ZF_CONN_USB-MICRO-B-SMD-holes" H 7050 5000 50  0001 C CNN
 F 3 "" H 7050 5000 50  0001 C CNN
 	1    6900 5050
@@
 $EndComp
 $Comp
-L GND #PWR01
+L GND #PWR21
 U 1 1 59441B12
 P 7900 2600
-F 0 "#PWR01" H 7900 2350 50  0001 C CNN
+F 0 "#PWR21" H 7900 2350 50  0001 C CNN
 F 1 "GND" H 7900 2450 50  0000 C CNN
 F 2 "" H 7900 2600 50  0001 C CNN
@@
 $EndComp
 $Comp
-L +3.3V #PWR02
+L +3.3V #PWR20
 U 1 1 59441B34
 P 7900 1900
-F 0 "#PWR02" H 7900 1750 50  0001 C CNN
+F 0 "#PWR20" H 7900 1750 50  0001 C CNN
 F 1 "+3.3V" H 7900 2040 50  0000 C CNN
 F 2 "" H 7900 1900 50  0001 C CNN
@@
 $EndComp
 $Comp
-L GND #PWR03
+L GND #PWR7
 U 1 1 59441B56
 P 3400 2350
-F 0 "#PWR03" H 3400 2100 50  0001 C CNN
+F 0 "#PWR7" H 3400 2100 50  0001 C CNN
 F 1 "GND" H 3400 2200 50  0000 C CNN
 F 2 "" H 3400 2350 50  0001 C CNN
@@
 A1IN
 $Comp
-L GND #PWR04
+L GND #PWR3
 U 1 1 59441D28
 P 1700 3800
-F 0 "#PWR04" H 1700 3550 50  0001 C CNN
+F 0 "#PWR3" H 1700 3550 50  0001 C CNN
 F 1 "GND" H 1700 3650 50  0000 C CNN
 F 2 "" H 1700 3800 50  0001 C CNN
@@
 $EndComp
 $Comp
-L GND #PWR05
+L GND #PWR1
 U 1 1 59441D70
 P 650 1150
-F 0 "#PWR05" H 650 900 50  0001 C CNN
+F 0 "#PWR1" H 650 900 50  0001 C CNN
 F 1 "GND" H 650 1000 50  0000 C CNN
 F 2 "" H 650 1150 50  0001 C CNN
@@
 $EndComp
 $Comp
-L GND #PWR06
+L GND #PWR8
 U 1 1 594424EB
 P 3450 1500
-F 0 "#PWR06" H 3450 1250 50  0001 C CNN
+F 0 "#PWR8" H 3450 1250 50  0001 C CNN
 F 1 "GND" H 3450 1350 50  0000 C CNN
 F 2 "" H 3450 1500 50  0001 C CNN
@@
 $EndComp
 $Comp
-L +3.3V #PWR07
+L +3.3V #PWR10
 U 1 1 594425F8
 P 4050 1150
-F 0 "#PWR07" H 4050 1000 50  0001 C CNN
+F 0 "#PWR10" H 4050 1000 50  0001 C CNN
 F 1 "+3.3V" H 4050 1290 50  0000 C CNN
 F 2 "" H 4050 1150 50  0001 C CNN
@@
 $EndComp
 $Comp
-L +3.3V #PWR08
+L +3.3V #PWR15
 U 1 1 594428AD
 P 7350 1100
-F 0 "#PWR08" H 7350 950 50  0001 C CNN
+F 0 "#PWR15" H 7350 950 50  0001 C CNN
 F 1 "+3.3V" H 7350 1240 50  0000 C CNN
 F 2 "" H 7350 1100 50  0001 C CNN
@@
 $EndComp
 $Comp
-L GND #PWR09
+L GND #PWR16
 U 1 1 59442909
 P 7350 3500
-F 0 "#PWR09" H 7350 3250 50  0001 C CNN
+F 0 "#PWR16" H 7350 3250 50  0001 C CNN
 F 1 "GND" H 7350 3350 50  0000 C CNN
 F 2 "" H 7350 3500 50  0001 C CNN
@@
 $EndComp
 $Comp
-L GND #PWR010
+L GND #PWR14
 U 1 1 59442B64
 P 6900 5850
-F 0 "#PWR010" H 6900 5600 50  0001 C CNN
+F 0 "#PWR14" H 6900 5600 50  0001 C CNN
 F 1 "GND" H 6900 5700 50  0000 C CNN
 F 2 "" H 6900 5850 50  0001 C CNN
@@
 $EndComp
 $Comp
-L GND #PWR011
+L GND #PWR13
 U 1 1 59442B8C
 P 6650 6100
-F 0 "#PWR011" H 6650 5850 50  0001 C CNN
+F 0 "#PWR13" H 6650 5850 50  0001 C CNN
 F 1 "GND" H 6650 5950 50  0000 C CNN
 F 2 "" H 6650 6100 50  0001 C CNN
@@
 $EndComp
 $Comp
-L +5V #PWR012
+L +5V #PWR17
 U 1 1 59442C78
 P 7350 4450
-F 0 "#PWR012" H 7350 4300 50  0001 C CNN
+F 0 "#PWR17" H 7350 4300 50  0001 C CNN
 F 1 "+5V" H 7350 4590 50  0000 C CNN
 F 2 "" H 7350 4450 50  0001 C CNN
@@
 F 0 "U3" H 8450 5750 50  0000 L CNN
 F 1 "FT230XQ" H 9300 5750 50  0000 L CNN
-F 2 "Housings_DFN_QFN:QFN-16-1EP_3x3mm_Pitch0.5mm" H 9000 5150 50  0001 C CNN
+F 2 "Housings_DFN_QFN:QFN-16-1EP_4x4mm_Pitch0.65mm" H 9000 5150 50  0001 C CNN
 F 3 "" H 9000 5150 50  0001 C CNN
 	1    9000 5150
@@
 	7350 4850 7200 4850
 $Comp
-L +3.3V #PWR013
+L +3.3V #PWR22
 U 1 1 594431FF
 P 8150 4250
-F 0 "#PWR013" H 8150 4100 50  0001 C CNN
+F 0 "#PWR22" H 8150 4100 50  0001 C CNN
 F 1 "+3.3V" H 8150 4390 50  0000 C CNN
 F 2 "" H 8150 4250 50  0001 C CNN
@@
 	8150 4250 8150 5350
 $Comp
-L +5V #PWR014
+L +5V #PWR23
 U 1 1 59443278
 P 8900 4200
-F 0 "#PWR014" H 8900 4050 50  0001 C CNN
+F 0 "#PWR23" H 8900 4050 50  0001 C CNN
 F 1 "+5V" H 8900 4340 50  0000 C CNN
 F 2 "" H 8900 4200 50  0001 C CNN
@@
 	8900 4450 8900 4200
 Text GLabel 6750 1550 2    60   Input ~ 0
+USART2_TX
+Text GLabel 6750 1400 2    60   Output ~ 0
 USART2_RX
-Text GLabel 6750 1400 2    60   Output ~ 0
-USART2_TX
 Wire Wire Line
 	6600 1400 6750 1400
@@
 	10000 4850 9700 4850
 $Comp
-L GND #PWR015
+L GND #PWR26
 U 1 1 594439C7
 P 9000 6100
-F 0 "#PWR015" H 9000 5850 50  0001 C CNN
+F 0 "#PWR26" H 9000 5850 50  0001 C CNN
 F 1 "GND" H 9000 5950 50  0000 C CNN
 F 2 "" H 9000 6100 50  0001 C CNN
@@
 $EndComp
 $Comp
-L +5V #PWR016
+L +5V #PWR5
 U 1 1 594446BF
 P 1900 5000
-F 0 "#PWR016" H 1900 4850 50  0001 C CNN
+F 0 "#PWR5" H 1900 4850 50  0001 C CNN
 F 1 "+5V" H 1900 5140 50  0000 C CNN
 F 2 "" H 1900 5000 50  0001 C CNN
@@
 $EndComp
 $Comp
-L +5VD #PWR017
+L +5VD #PWR9
 U 1 1 594447B7
 P 4000 5000
-F 0 "#PWR017" H 4000 4850 50  0001 C CNN
+F 0 "#PWR9" H 4000 4850 50  0001 C CNN
 F 1 "+5VD" H 4000 5140 50  0000 C CNN
 F 2 "" H 4000 5000 50  0001 C CNN
@@
 $EndComp
 $Comp
-L GND #PWR018
+L GND #PWR6
 U 1 1 59444A62
 P 2000 5800
-F 0 "#PWR018" H 2000 5550 50  0001 C CNN
+F 0 "#PWR6" H 2000 5550 50  0001 C CNN
 F 1 "GND" H 2000 5650 50  0000 C CNN
 F 2 "" H 2000 5800 50  0001 C CNN
@@
 $EndComp
 $Comp
-L GND #PWR019
+L GND #PWR12
 U 1 1 59444CB7
 P 4950 5900
-F 0 "#PWR019" H 4950 5650 50  0001 C CNN
+F 0 "#PWR12" H 4950 5650 50  0001 C CNN
 F 1 "GND" H 4950 5750 50  0000 C CNN
 F 2 "" H 4950 5900 50  0001 C CNN
@@
 Connection ~ 4250 5550
 $Comp
-L +5V #PWR020
+L +5V #PWR11
 U 1 1 5944518C
 P 4250 4850
-F 0 "#PWR020" H 4250 4700 50  0001 C CNN
+F 0 "#PWR11" H 4250 4700 50  0001 C CNN
 F 1 "+5V" H 4250 4990 50  0000 C CNN
 F 2 "" H 4250 4850 50  0001 C CNN
@@
 	4250 4850 4250 4950
 $Comp
-L +5VD #PWR021
+L +5VD #PWR4
 U 1 1 594452E4
 P 1800 2000
-F 0 "#PWR021" H 1800 1850 50  0001 C CNN
+F 0 "#PWR4" H 1800 1850 50  0001 C CNN
 F 1 "+5VD" H 1800 2140 50  0000 C CNN
 F 2 "" H 1800 2000 50  0001 C CNN
@@
 $EndComp
 $Comp
-L +5V #PWR022
+L +5V #PWR24
 U 1 1 5946EA88
-P 8750 1900
-F 0 "#PWR022" H 8750 1750 50  0001 C CNN
-F 1 "+5V" H 8750 2040 50  0000 C CNN
-F 2 "" H 8750 1900 50  0001 C CNN
-F 3 "" H 8750 1900 50  0001 C CNN
-	1    8750 1900
-	1    0    0    -1
-$EndComp
-$Comp
-L GND #PWR023
+P 9000 1900
+F 0 "#PWR24" H 9000 1750 50  0001 C CNN
+F 1 "+5V" H 9000 2040 50  0000 C CNN
+F 2 "" H 9000 1900 50  0001 C CNN
+F 3 "" H 9000 1900 50  0001 C CNN
+	1    9000 1900
+	1    0    0    -1
+$EndComp
+$Comp
+L GND #PWR25
 U 1 1 5946EB1C
-P 8750 2550
-F 0 "#PWR023" H 8750 2300 50  0001 C CNN
-F 1 "GND" H 8750 2400 50  0000 C CNN
-F 2 "" H 8750 2550 50  0001 C CNN
-F 3 "" H 8750 2550 50  0001 C CNN
-	1    8750 2550
-	1    0    0    -1
-$EndComp
-Wire Wire Line
-	8750 1900 8750 2050
-Wire Wire Line
-	8750 2350 8750 2550
+P 9000 2550
+F 0 "#PWR25" H 9000 2300 50  0001 C CNN
+F 1 "GND" H 9000 2400 50  0000 C CNN
+F 2 "" H 9000 2550 50  0001 C CNN
+F 3 "" H 9000 2550 50  0001 C CNN
+	1    9000 2550
+	1    0    0    -1
+$EndComp
 Wire Wire Line
 	7200 5050 7600 5050
@@
 Connection ~ 7550 5150
 $Comp
-L GND #PWR024
+L GND #PWR18
 U 1 1 5946F3F4
 P 7350 6000
-F 0 "#PWR024" H 7350 5750 50  0001 C CNN
+F 0 "#PWR18" H 7350 5750 50  0001 C CNN
 F 1 "GND" H 7350 5850 50  0000 C CNN
 F 2 "" H 7350 6000 50  0001 C CNN
@@
 $EndComp
 $Comp
-L GND #PWR025
+L GND #PWR19
 U 1 1 5946F430
 P 7550 6000
-F 0 "#PWR025" H 7550 5750 50  0001 C CNN
+F 0 "#PWR19" H 7550 5750 50  0001 C CNN
 F 1 "GND" H 7550 5850 50  0000 C CNN
 F 2 "" H 7550 6000 50  0001 C CNN
@@
 $EndComp
 $Comp
-L GND #PWR026
+L GND #PWR2
 U 1 1 59472434
 P 1700 1500
-F 0 "#PWR026" H 1700 1250 50  0001 C CNN
+F 0 "#PWR2" H 1700 1250 50  0001 C CNN
 F 1 "GND" H 1700 1350 50  0000 C CNN
 F 2 "" H 1700 1500 50  0001 C CNN
@@
 Wire Wire Line
 	4200 3350 4000 3350
+$Comp
+L C C9
+U 1 1 5947E653
+P 9000 2200
+F 0 "C9" H 9025 2300 50  0000 L CNN
+F 1 "C" H 9025 2100 50  0000 L CNN
+F 2 "ZF_footprints:ZF_SMD_NonPol_0402_cap" H 9038 2050 50  0001 C CNN
+F 3 "" H 9000 2200 50  0001 C CNN
+	1    9000 2200
+	1    0    0    -1
+$EndComp
+$Comp
+L C C10
+U 1 1 5947E698
+P 9250 2200
+F 0 "C10" H 9275 2300 50  0000 L CNN
+F 1 "C" H 9275 2100 50  0000 L CNN
+F 2 "ZF_footprints:ZF_SMD_NonPol_0402_cap" H 9288 2050 50  0001 C CNN
+F 3 "" H 9250 2200 50  0001 C CNN
+	1    9250 2200
+	1    0    0    -1
+$EndComp
+Wire Wire Line
+	8750 2050 9250 2050
+Connection ~ 9000 2050
+Wire Wire Line
+	8750 2350 9250 2350
+Connection ~ 9000 2350
+Wire Wire Line
+	9000 1900 9000 2050
+Wire Wire Line
+	9000 2350 9000 2550
 $EndSCHEMATC

Commit message: fixed pcb
Parts:
- C10: value C -> 4.7uF; footprint ZF_footprints:ZF_SMD_NonPol_0402_cap -> Resistors_SMD:R_0603_HandSoldering
Changed lines of the file:
@@
 $EndComp
 $Comp
-L GND #PWR21
+L GND #PWR01
 U 1 1 59441B12
 P 7900 2600
-F 0 "#PWR21" H 7900 2350 50  0001 C CNN
+F 0 "#PWR01" H 7900 2350 50  0001 C CNN
 F 1 "GND" H 7900 2450 50  0000 C CNN
 F 2 "" H 7900 2600 50  0001 C CNN
@@
 $EndComp
 $Comp
-L +3.3V #PWR20
+L +3.3V #PWR02
 U 1 1 59441B34
 P 7900 1900
-F 0 "#PWR20" H 7900 1750 50  0001 C CNN
+F 0 "#PWR02" H 7900 1750 50  0001 C CNN
 F 1 "+3.3V" H 7900 2040 50  0000 C CNN
 F 2 "" H 7900 1900 50  0001 C CNN
@@
 $EndComp
 $Comp
-L GND #PWR7
+L GND #PWR03
 U 1 1 59441B56
 P 3400 2350
-F 0 "#PWR7" H 3400 2100 50  0001 C CNN
+F 0 "#PWR03" H 3400 2100 50  0001 C CNN
 F 1 "GND" H 3400 2200 50  0000 C CNN
 F 2 "" H 3400 2350 50  0001 C CNN
@@
 A1IN
 $Comp
-L GND #PWR3
+L GND #PWR04
 U 1 1 59441D28
 P 1700 3800
-F 0 "#PWR3" H 1700 3550 50  0001 C CNN
+F 0 "#PWR04" H 1700 3550 50  0001 C CNN
 F 1 "GND" H 1700 3650 50  0000 C CNN
 F 2 "" H 1700 3800 50  0001 C CNN
@@
 $EndComp
 $Comp
-L GND #PWR1
+L GND #PWR05
 U 1 1 59441D70
 P 650 1150
-F 0 "#PWR1" H 650 900 50  0001 C CNN
+F 0 "#PWR05" H 650 900 50  0001 C CNN
 F 1 "GND" H 650 1000 50  0000 C CNN
 F 2 "" H 650 1150 50  0001 C CNN
@@
 $EndComp
 $Comp
-L GND #PWR8
+L GND #PWR06
 U 1 1 594424EB
 P 3450 1500
-F 0 "#PWR8" H 3450 1250 50  0001 C CNN
+F 0 "#PWR06" H 3450 1250 50  0001 C CNN
 F 1 "GND" H 3450 1350 50  0000 C CNN
 F 2 "" H 3450 1500 50  0001 C CNN
@@
 $EndComp
 $Comp
-L +3.3V #PWR10
+L +3.3V #PWR07
 U 1 1 594425F8
 P 4050 1150
-F 0 "#PWR10" H 4050 1000 50  0001 C CNN
+F 0 "#PWR07" H 4050 1000 50  0001 C CNN
 F 1 "+3.3V" H 4050 1290 50  0000 C CNN
 F 2 "" H 4050 1150 50  0001 C CNN
@@
 $EndComp
 $Comp
-L +3.3V #PWR15
+L +3.3V #PWR08
 U 1 1 594428AD
 P 7350 1100
-F 0 "#PWR15" H 7350 950 50  0001 C CNN
+F 0 "#PWR08" H 7350 950 50  0001 C CNN
 F 1 "+3.3V" H 7350 1240 50  0000 C CNN
 F 2 "" H 7350 1100 50  0001 C CNN
@@
 $EndComp
 $Comp
-L GND #PWR16
+L GND #PWR09
 U 1 1 59442909
 P 7350 3500
-F 0 "#PWR16" H 7350 3250 50  0001 C CNN
+F 0 "#PWR09" H 7350 3250 50  0001 C CNN
 F 1 "GND" H 7350 3350 50  0000 C CNN
 F 2 "" H 7350 3500 50  0001 C CNN
@@
 $EndComp
 $Comp
-L GND #PWR14
+L GND #PWR010
 U 1 1 59442B64
 P 6900 5850
-F 0 "#PWR14" H 6900 5600 50  0001 C CNN
+F 0 "#PWR010" H 6900 5600 50  0001 C CNN
 F 1 "GND" H 6900 5700 50  0000 C CNN
 F 2 "" H 6900 5850 50  0001 C CNN
@@
 $EndComp
 $Comp
-L GND #PWR13
+L GND #PWR011
 U 1 1 59442B8C
 P 6650 6100
-F 0 "#PWR13" H 6650 5850 50  0001 C CNN
+F 0 "#PWR011" H 6650 5850 50  0001 C CNN
 F 1 "GND" H 6650 5950 50  0000 C CNN
 F 2 "" H 6650 6100 50  0001 C CNN
@@
 $EndComp
 $Comp
-L +5V #PWR17
+L +5V #PWR012
 U 1 1 59442C78
 P 7350 4450
-F 0 "#PWR17" H 7350 4300 50  0001 C CNN
+F 0 "#PWR012" H 7350 4300 50  0001 C CNN
 F 1 "+5V" H 7350 4590 50  0000 C CNN
 F 2 "" H 7350 4450 50  0001 C CNN
@@
 	7350 4850 7200 4850
 $Comp
-L +3.3V #PWR22
+L +3.3V #PWR013
 U 1 1 594431FF
 P 8150 4250
-F 0 "#PWR22" H 8150 4100 50  0001 C CNN
+F 0 "#PWR013" H 8150 4100 50  0001 C CNN
 F 1 "+3.3V" H 8150 4390 50  0000 C CNN
 F 2 "" H 8150 4250 50  0001 C CNN
@@
 	8150 4250 8150 5350
 $Comp
-L +5V #PWR23
+L +5V #PWR014
 U 1 1 59443278
 P 8900 4200
-F 0 "#PWR23" H 8900 4050 50  0001 C CNN
+F 0 "#PWR014" H 8900 4050 50  0001 C CNN
 F 1 "+5V" H 8900 4340 50  0000 C CNN
 F 2 "" H 8900 4200 50  0001 C CNN
@@
 	10000 4850 9700 4850
 $Comp
-L GND #PWR26
+L GND #PWR015
 U 1 1 594439C7
 P 9000 6100
-F 0 "#PWR26" H 9000 5850 50  0001 C CNN
+F 0 "#PWR015" H 9000 5850 50  0001 C CNN
 F 1 "GND" H 9000 5950 50  0000 C CNN
 F 2 "" H 9000 6100 50  0001 C CNN
@@
 $EndComp
 $Comp
-L +5V #PWR5
+L +5V #PWR016
 U 1 1 594446BF
 P 1900 5000
-F 0 "#PWR5" H 1900 4850 50  0001 C CNN
+F 0 "#PWR016" H 1900 4850 50  0001 C CNN
 F 1 "+5V" H 1900 5140 50  0000 C CNN
 F 2 "" H 1900 5000 50  0001 C CNN
@@
 $EndComp
 $Comp
-L +5VD #PWR9
+L +5VD #PWR017
 U 1 1 594447B7
 P 4000 5000
-F 0 "#PWR9" H 4000 4850 50  0001 C CNN
+F 0 "#PWR017" H 4000 4850 50  0001 C CNN
 F 1 "+5VD" H 4000 5140 50  0000 C CNN
 F 2 "" H 4000 5000 50  0001 C CNN
@@
 $EndComp
 $Comp
-L GND #PWR6
+L GND #PWR018
 U 1 1 59444A62
 P 2000 5800
-F 0 "#PWR6" H 2000 5550 50  0001 C CNN
+F 0 "#PWR018" H 2000 5550 50  0001 C CNN
 F 1 "GND" H 2000 5650 50  0000 C CNN
 F 2 "" H 2000 5800 50  0001 C CNN
@@
 $EndComp
 $Comp
-L GND #PWR12
+L GND #PWR019
 U 1 1 59444CB7
 P 4950 5900
-F 0 "#PWR12" H 4950 5650 50  0001 C CNN
+F 0 "#PWR019" H 4950 5650 50  0001 C CNN
 F 1 "GND" H 4950 5750 50  0000 C CNN
 F 2 "" H 4950 5900 50  0001 C CNN
@@
 Connection ~ 4250 5550
 $Comp
-L +5V #PWR11
+L +5V #PWR020
 U 1 1 5944518C
 P 4250 4850
-F 0 "#PWR11" H 4250 4700 50  0001 C CNN
+F 0 "#PWR020" H 4250 4700 50  0001 C CNN
 F 1 "+5V" H 4250 4990 50  0000 C CNN
 F 2 "" H 4250 4850 50  0001 C CNN
@@
 	4250 4850 4250 4950
 $Comp
-L +5VD #PWR4
+L +5VD #PWR021
 U 1 1 594452E4
 P 1800 2000
-F 0 "#PWR4" H 1800 1850 50  0001 C CNN
+F 0 "#PWR021" H 1800 1850 50  0001 C CNN
 F 1 "+5VD" H 1800 2140 50  0000 C CNN
 F 2 "" H 1800 2000 50  0001 C CNN
@@
 $EndComp
 $Comp
-L +5V #PWR24
+L +5V #PWR022
 U 1 1 5946EA88
 P 9000 1900
-F 0 "#PWR24" H 9000 1750 50  0001 C CNN
+F 0 "#PWR022" H 9000 1750 50  0001 C CNN
 F 1 "+5V" H 9000 2040 50  0000 C CNN
 F 2 "" H 9000 1900 50  0001 C CNN
@@
 $EndComp
 $Comp
-L GND #PWR25
+L GND #PWR023
 U 1 1 5946EB1C
 P 9000 2550
-F 0 "#PWR25" H 9000 2300 50  0001 C CNN
+F 0 "#PWR023" H 9000 2300 50  0001 C CNN
 F 1 "GND" H 9000 2400 50  0000 C CNN
 F 2 "" H 9000 2550 50  0001 C CNN
@@
 Connection ~ 7550 5150
 $Comp
-L GND #PWR18
+L GND #PWR024
 U 1 1 5946F3F4
 P 7350 6000
-F 0 "#PWR18" H 7350 5750 50  0001 C CNN
+F 0 "#PWR024" H 7350 5750 50  0001 C CNN
 F 1 "GND" H 7350 5850 50  0000 C CNN
 F 2 "" H 7350 6000 50  0001 C CNN
@@
 $EndComp
 $Comp
-L GND #PWR19
+L GND #PWR025
 U 1 1 5946F430
 P 7550 6000
-F 0 "#PWR19" H 7550 5750 50  0001 C CNN
+F 0 "#PWR025" H 7550 5750 50  0001 C CNN
 F 1 "GND" H 7550 5850 50  0000 C CNN
 F 2 "" H 7550 6000 50  0001 C CNN
@@
 $EndComp
 $Comp
-L GND #PWR2
+L GND #PWR026
 U 1 1 59472434
 P 1700 1500
-F 0 "#PWR2" H 1700 1250 50  0001 C CNN
+F 0 "#PWR026" H 1700 1250 50  0001 C CNN
 F 1 "GND" H 1700 1350 50  0000 C CNN
 F 2 "" H 1700 1500 50  0001 C CNN
@@
 P 9250 2200
 F 0 "C10" H 9275 2300 50  0000 L CNN
-F 1 "C" H 9275 2100 50  0000 L CNN
-F 2 "ZF_footprints:ZF_SMD_NonPol_0402_cap" H 9288 2050 50  0001 C CNN
+F 1 "4.7uF" H 9275 2100 50  0000 L CNN
+F 2 "Resistors_SMD:R_0603_HandSoldering" H 9288 2050 50  0001 C CNN
 F 3 "" H 9250 2200 50  0001 C CNN
 	1    9250 2200
