File: HARDWARE/4-layer/NeuroBytes_NID_4-layer.kicad_pcb (KiCad board)
At the start: 4 copper layers, 46 x 45 mm, 64 parts, among them J1 CONN_01X05, J3 USB_OTG, Q1 MMBT3904, Q2 2N7002, U1 TPS2550, U2 STM32F103CBUx, U3 LD3985G, U4 RClamp0503F, Y1 8 MHz

Commit message: updates to 4-layer and enclosed NID versions
Other:
- board text removed: "COMPONENT POSITION ORIGIN"
- board text removed: "INSTALL FOUR POLYURETHANE BUMPERS IN FOUR 10MM SILKSCREEN CIRCLES (BACK)"
- board text removed: "NOTES: 1. FOOTPRINTS ORIENTED PER IPC-7351FC LEVEL B (PIN 1 IN LOWER LEFT) 2. COMPONENT ROTATION IN DEGREES COUNTER-CLOCKWISE 3. COMPONENTS MOUNTED ON BOTH SIDES (FOUR LEDS ON FRONT, ALL OTHERS ON BACK) 4. PCB IS 1.6mm FR4 RATED FOR ROHS REFLOW, 1OZ COPPER, ENIG FINISH 5. MATTE BLACK SOLDER MASK WITH WHITE SILKSCREEN 6. SOLDER PASTE MUST BE ROHS COMPLIANT (LEAD-FREE) 7. NO MARKS (E-TEST, QA, SERI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"
Changed lines of the file:
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@@
     (area 56.399999 45.025 221.600001 145.325)
     (thickness 1.6)
-    (drawings 117)
+    (drawings 106)
     (tracks 499)
     (zones 0)
@@
   )
   (setup
-    (last_trace_width 0.35)
+    (last_trace_width 0.2)
     (user_trace_width 0.35)
     (user_trace_width 0.5)
@@
   (gr_line (start 149.5 86.5) (end 149.5 86.5) (layer F.Fab) (width 0.2))
   (gr_line (start 149.5 88.5) (end 149.5 86.5) (layer F.Fab) (width 0.2))
-  (gr_line (start 157.5 80.5) (end 149.5 88.5) (layer F.Fab) (width 0.2))
-  (gr_line (start 157.5 70.5) (end 157.5 80.5) (layer F.Fab) (width 0.2))
   (gr_line (start 144.5 66.5) (end 146.5 66.5) (layer F.Fab) (width 0.2))
   (gr_line (start 221.5 70.5) (end 221.5 70.5) (layer F.Fab) (width 0.2))
-  (gr_line (start 148.5 70.5) (end 221.5 70.5) (layer F.Fab) (width 0.2))
-  (gr_line (start 144.5 66.5) (end 148.5 70.5) (layer F.Fab) (width 0.2))
-  (gr_line (start 106.5 106.5) (end 145.5 106.5) (layer F.Fab) (width 0.2))
   (gr_line (start 106.5 106.5) (end 106.5 106.5) (layer F.Fab) (width 0.2))
-  (gr_line (start 103.5 103.5) (end 106.5 106.5) (layer F.Fab) (width 0.2))
-  (gr_line (start 100.5 102.5) (end 104.5 102.5) (layer F.Fab) (width 0.2))
-  (gr_line (start 102.5 100.5) (end 102.5 104.5) (layer F.Fab) (width 0.2))
   (gr_line (start 148.5 60.5) (end 150.5 60.5) (layer F.Fab) (width 0.2))
   (gr_line (start 148.5 58.5) (end 148.5 58.5) (layer F.Fab) (width 0.2))
@@
   (gr_line (start 152.5 91.5) (end 154.5 89.5) (layer F.Fab) (width 0.2))
   (gr_line (start 195.5 91.5) (end 152.5 91.5) (layer F.Fab) (width 0.2))
-  (gr_text "INSTALL FOUR POLYURETHANE BUMPERS\nIN FOUR 10MM SILKSCREEN CIRCLES (BACK)" (at 195.5 67.5) (layer F.Fab)
-    (effects (font (size 1.5 1.5) (thickness 0.3)))
-  )
-  (gr_text "NOTES:\n1. FOOTPRINTS ORIENTED PER IPC-7351FC LEVEL B (PIN 1 IN LOWER LEFT)\n2. COMPONENT ROTATION IN DEGREES COUNTER-CLOCKWISE\n3. COMPONENTS MOUNTED ON BOTH SIDES (FOUR LEDS ON FRONT, ALL OTHERS ON BACK)\n4. PCB IS 1.6mm FR4 RATED FOR ROHS REFLOW, 1OZ COPPER, ENIG FINISH\n5. MATTE BLACK SOLDER MASK WITH WHITE SILKSCREEN\n6. SOLDER PASTE MUST BE ROHS COMPLIANT (LEAD-FREE)\n7. NO MARKS (E-TEST, QA, SERIAL NUMBER, ETC) ON FRONT (LOGO SIDE) OF BOARD\n8. BOARDS TO BE SHIPPED IN INDIVIDUAL ANTI-STATIC BAGS\n9. FOUR SELF-ADHESIVE POLYURETHANE BUMPERS TO BE APPLIED AS SHOWN AFTER ASSEMBLY" (at 88.5 132.5) (layer F.Fab)
-    (effects (font (size 1.5 1.5) (thickness 0.3)) (justify left))
-  )
-  (gr_text "COMPONENT POSITION ORIGIN" (at 127.5 105) (layer F.Fab)
-    (effects (font (size 1.5 1.5) (thickness 0.3)))
-  )
   (gr_text "V-SCORE PARALLEL SIDES" (at 72.5 90) (layer F.Fab)
     (effects (font (size 1.5 1.5) (thickness 0.3)))
@@
   (segment (start 119.024264 83) (end 119.024264 81.703301) (width 0.2) (layer B.Cu) (net 3))
   (segment (start 119.024264 81.703301) (end 119.131371 81.596194) (width 0.2) (layer B.Cu) (net 3))
-  (segment (start 124.548528 85.224264) (end 124.55 85.224264) (width 0.35) (layer B.Cu) (net 4) (status C00000))
-  (segment (start 124.55 85.224264) (end 125.374264 84.4) (width 0.35) (layer B.Cu) (net 4) (status 400000))
+  (segment (start 124.548528 85.224264) (end 124.55 85.224264) (width 0.35) (layer B.Cu) (net 4))
+  (segment (start 124.55 85.224264) (end 125.374264 84.4) (width 0.35) (layer B.Cu) (net 4))
   (segment (start 125.374264 84.4) (end 125.374264 84.369963) (width 0.35) (layer B.Cu) (net 4))
   (segment (start 128.17064 90.923624) (end 128.17064 89.15) (width 0.35) (layer B.Cu) (net 4))
