File: HARDWARE/Enclosed/NeuroBytes_NID_Enclosed.kicad_pcb (KiCad board)
At the start: 2 copper layers, 40.6 x 72.2 mm, 74 parts, among them J1 CONN_01X05, J2 Conn_01x03, J3 USB_OTG, J4 Conn_01x03_Female, J5 Conn_01x03, J6 Conn_01x03_Female, J7 Conn_01x03, J8 Conn_01x03_Female, Q1 MMBT3904, Q2 2N7002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

Commit message: updates to 4-layer and enclosed NID versions
Routing:
- net (no net): track 4.27 -> 0.00 mm, vias 2 -> 0
Changed lines of the file:
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@@
     (links 153)
     (no_connects 0)
-    (area 25.974263 44.949998 66.674265 117.250001)
+    (area 21.448549 37.5 221.600001 145.325)
     (thickness 1.6)
     (drawings 103)
-    (tracks 623)
+    (tracks 618)
     (zones 0)
     (modules 74)
@@
     (effects (font (size 1.5 1.5) (thickness 0.21)))
   )
-  (segment (start 44.624264 46.25) (end 48.424264 46.25) (width 0.2) (layer B.Cu) (net 0))
-  (segment (start 48.424264 46.25) (end 48.524264 46.35) (width 0.2) (layer B.Cu) (net 0))
-  (via (at 48.524264 46.35) (size 0.6) (drill 0.4) (layers F.Cu B.Cu) (net 0))
-  (segment (start 44.38934 46.484924) (end 44.624264 46.25) (width 0.2) (layer F.Cu) (net 0))
-  (via (at 44.624264 46.25) (size 0.6) (drill 0.4) (layers F.Cu B.Cu) (net 0))
   (segment (start 53.224264 53.35) (end 54.124264 54.25) (width 0.2) (layer F.Cu) (net 1))
   (segment (start 54.124264 54.25) (end 57.724264 54.25) (width 0.2) (layer F.Cu) (net 1))
